Commit message: chore: publish lab cobot workspace

File: src/lab_cobot_description/urdf/inc/mecanum_base.xacro (robot description, xacro)
@@ -35,5 +35,5 @@
     </joint>
     <!-- 4 个麦轮(纯视觉装饰) -->
-    <xacro:macro name="mec_wheel" params="name x y">
+    <xacro:macro name="mec_wheel" params="name x y roller_slant">
       <link name="${name}">
         <visual>
@@ -41,4 +41,56 @@
           <geometry><cylinder radius="${wheel_radius}" length="${wheel_width}"/></geometry>
           <material name="wheel_dark"><color rgba="0.10 0.10 0.10 1.0"/></material>
+        </visual>
+        <!-- Side-face roller strips make the wheels read as mecanum in Gazebo/RViz
+             while keeping the wheel collision-free for planar_move. -->
+        <visual name="${name}_roller_outer_0">
+          <origin xyz="0 ${wheel_width/2.0 + 0.003} ${-wheel_radius*0.46}" rpy="0 ${roller_slant*pi/4.0} 0"/>
+          <geometry><box size="${wheel_radius*1.45} 0.006 0.012"/></geometry>
+          <material name="roller_light"><color rgba="0.62 0.66 0.68 1.0"/></material>
+        </visual>
+        <visual name="${name}_roller_outer_1">
+          <origin xyz="0 ${wheel_width/2.0 + 0.003} ${-wheel_radius*0.23}" rpy="0 ${roller_slant*pi/4.0} 0"/>
+          <geometry><box size="${wheel_radius*1.45} 0.006 0.012"/></geometry>
+          <material name="roller_light"><color rgba="0.62 0.66 0.68 1.0"/></material>
+        </visual>
+        <visual name="${name}_roller_outer_2">
+          <origin xyz="0 ${wheel_width/2.0 + 0.003} 0" rpy="0 ${roller_slant*pi/4.0} 0"/>
+          <geometry><box size="${wheel_radius*1.45} 0.006 0.012"/></geometry>
+          <material name="roller_light"><color rgba="0.62 0.66 0.68 1.0"/></material>
+        </visual>
+        <visual name="${name}_roller_outer_3">
+          <origin xyz="0 ${wheel_width/2.0 + 0.003} ${wheel_radius*0.23}" rpy="0 ${roller_slant*pi/4.0} 0"/>
+          <geometry><box size="${wheel_radius*1.45} 0.006 0.012"/></geometry>
+          <material name="roller_light"><color rgba="0.62 0.66 0.68 1.0"/></material>
+        </visual>
+        <visual name="${name}_roller_outer_4">
+          <origin xyz="0 ${wheel_width/2.0 + 0.003} ${wheel_radius*0.46}" rpy="0 ${roller_slant*pi/4.0} 0"/>
+          <geometry><box size="${wheel_radius*1.45} 0.006 0.012"/></geometry>
+          <material name="roller_light"><color rgba="0.62 0.66 0.68 1.0"/></material>
+        </visual>
+        <visual name="${name}_roller_inner_0">
+          <origin xyz="0 ${-(wheel_width/2.0 + 0.003)} ${-wheel_radius*0.46}" rpy="0 ${roller_slant*pi/4.0} 0"/>
+          <geometry><box size="${wheel_radius*1.45} 0.006 0.012"/></geometry>
+          <material name="roller_light"><color rgba="0.62 0.66 0.68 1.0"/></material>
+        </visual>
+        <visual name="${name}_roller_inner_1">
+          <origin xyz="0 ${-(wheel_width/2.0 + 0.003)} ${-wheel_radius*0.23}" rpy="0 ${roller_slant*pi/4.0} 0"/>
+          <geometry><box size="${wheel_radius*1.45} 0.006 0.012"/></geometry>
+          <material name="roller_light"><color rgba="0.62 0.66 0.68 1.0"/></material>
+        </visual>
+        <visual name="${name}_roller_inner_2">
+          <origin xyz="0 ${-(wheel_width/2.0 + 0.003)} 0" rpy="0 ${roller_slant*pi/4.0} 0"/>
+          <geometry><box size="${wheel_radius*1.45} 0.006 0.012"/></geometry>
+          <material name="roller_light"><color rgba="0.62 0.66 0.68 1.0"/></material>
+        </visual>
+        <visual name="${name}_roller_inner_3">
+          <origin xyz="0 ${-(wheel_width/2.0 + 0.003)} ${wheel_radius*0.23}" rpy="0 ${roller_slant*pi/4.0} 0"/>
+          <geometry><box size="${wheel_radius*1.45} 0.006 0.012"/></geometry>
+          <material name="roller_light"><color rgba="0.62 0.66 0.68 1.0"/></material>
+        </visual>
+        <visual name="${name}_roller_inner_4">
+          <origin xyz="0 ${-(wheel_width/2.0 + 0.003)} ${wheel_radius*0.46}" rpy="0 ${roller_slant*pi/4.0} 0"/>
+          <geometry><box size="${wheel_radius*1.45} 0.006 0.012"/></geometry>
+          <material name="roller_light"><color rgba="0.62 0.66 0.68 1.0"/></material>
         </visual>
         <xacro:cylinder_inertia m="1.2" r="${wheel_radius}" l="${wheel_width}"/>
@@ -52,8 +104,8 @@
       <gazebo reference="${name}"><material>Gazebo/FlatBlack</material></gazebo>
     </xacro:macro>
-    <xacro:mec_wheel name="wheel_fl" x="${wx}"  y="${wy}"/>
-    <xacro:mec_wheel name="wheel_fr" x="${wx}"  y="${-wy}"/>
-    <xacro:mec_wheel name="wheel_rl" x="${-wx}" y="${wy}"/>
-    <xacro:mec_wheel name="wheel_rr" x="${-wx}" y="${-wy}"/>
+    <xacro:mec_wheel name="wheel_fl" x="${wx}"  y="${wy}"  roller_slant="1"/>
+    <xacro:mec_wheel name="wheel_fr" x="${wx}"  y="${-wy}" roller_slant="-1"/>
+    <xacro:mec_wheel name="wheel_rl" x="${-wx}" y="${wy}"  roller_slant="-1"/>
+    <xacro:mec_wheel name="wheel_rr" x="${-wx}" y="${-wy}" roller_slant="1"/>
     <!-- 全向驱动插件:订阅 /cmd_vel(Twist 全向),发布 /odom -->
     <gazebo>

File: src/lab_cobot_description/urdf/inc/sensors.xacro (robot description, xacro)
@@ -72,9 +72,9 @@
       <xacro:box_inertia m="0.05" x="0.03" y="0.09" z="0.025"/>
     </link>
-    <!-- 装在立柱上方、向前下俯视(pitch 向下 0.5rad) -->
+    <!-- 装在立柱上方、略高于桌面，向前轻微俯视 station_a 样件 -->
     <joint name="camera_joint" type="fixed">
       <parent link="arm_mount_link"/>
       <child link="camera_link"/>
-      <origin xyz="0.10 0 0.05" rpy="0 0.5 0"/>
+      <origin xyz="0.10 0 0.35" rpy="0 0.15 0"/>
     </joint>
     <!-- 光学系(REP-103:z 向前,x 向右,y 向下) -->

File: src/lab_cobot_description/urdf/inc/vacuum_gripper.xacro (robot description, xacro)
@@ -27,4 +27,7 @@
       <origin xyz="0 0 0" rpy="0 0 0"/>
     </joint>
+    <gazebo reference="suction_joint">
+      <preserveFixedJoint>true</preserveFixedJoint>
+    </gazebo>
     <!-- 吸附作用点(TCP 末端) -->
     <link name="grasp_point"/>
@@ -34,5 +37,8 @@
       <origin xyz="0 0 0.04" rpy="0 0 0"/>
     </joint>
-    <gazebo reference="suction_link"><material>Gazebo/Red</material></gazebo>
+    <gazebo reference="suction_link">
+      <material>Gazebo/Red</material>
+      <preserveFixedJoint>true</preserveFixedJoint>
+    </gazebo>
     <!-- 真空吸盘插件:service /suction/switch(std_srvs/SetBool)开关,
          topic /suction/grasping(std_msgs/Bool)状态。max_distance 内的非 fixed 物体被吸附。 -->
@@ -44,5 +50,5 @@
           <remapping>grasping:=suction/grasping</remapping>
         </ros>
-        <link_name>suction_link</link_name>
+        <link_name>ur_wrist_3_link</link_name>
         <max_distance>0.06</max_distance>
         <fixed>ground_plane</fixed>

File: src/lab_cobot_description/urdf/lab_cobot.urdf.xacro (robot description, xacro)
@@ -1,5 +1,5 @@
 <?xml version="1.0"?>
 <!--
-  一体化麦轮移动机械臂:麦轮全向底盘 + 基座立柱 + UR5e + 真空吸盘 + 传感器。
+  一体化麦轮移动机械臂:麦轮全向底盘 + 基座立柱 + UR5e + 平行夹爪 + 传感器。
   UR5e 用官方 ur_description 的 ur_robot macro(sim_gazebo 模式),装在立柱顶 arm_mount_link。
   关节由 gazebo_ros2_control 驱动;底盘由 gazebo_ros_planar_move 驱动。
@@ -18,5 +18,5 @@
   <xacro:include filename="$(find lab_cobot_description)/urdf/inc/pillar.xacro"/>
   <xacro:include filename="$(find lab_cobot_description)/urdf/inc/sensors.xacro"/>
-  <xacro:include filename="$(find lab_cobot_description)/urdf/inc/vacuum_gripper.xacro"/>
+  <xacro:include filename="$(find lab_cobot_description)/urdf/inc/parallel_gripper.xacro"/>
   <!-- ===== UR5e 参数 ===== -->
   <xacro:arg name="ur_type" default="ur5e"/>
@@ -76,6 +76,59 @@
     <origin xyz="0 0 0" rpy="0 0 0"/>
   </xacro:ur_robot>
-  <!-- ===== 末端真空吸盘(挂 UR tool0,带 tf_prefix) ===== -->
-  <xacro:vacuum_gripper parent="ur_tool0"/>
+  <!-- ===== Parallel gripper mounted on UR tool0 ===== -->
+  <xacro:parallel_gripper parent="ur_tool0"/>
+  <ros2_control name="gripper_and_wheel_visuals" type="system">
+    <hardware>
+      <plugin>gazebo_ros2_control/GazeboSystem</plugin>
+    </hardware>
+    <joint name="gripper_left_finger_joint">
+      <command_interface name="position"/>
+      <state_interface name="position">
+        <param name="initial_value">0.0</param>
+      </state_interface>
+      <state_interface name="velocity"/>
+      <state_interface name="effort"/>
+    </joint>
+    <joint name="gripper_right_finger_joint">
+      <command_interface name="position"/>
+      <state_interface name="position">
+        <param name="initial_value">0.0</param>
+      </state_interface>
+      <state_interface name="velocity"/>
+      <state_interface name="effort"/>
+    </joint>
+    <joint name="wheel_fl_joint">
+      <command_interface name="velocity"/>
+      <state_interface name="position">
+        <param name="initial_value">0.0</param>
+      </state_interface>
+      <state_interface name="velocity"/>
+      <state_interface name="effort"/>
+    </joint>
+    <joint name="wheel_fr_joint">
+      <command_interface name="velocity"/>
+      <state_interface name="position">
+        <param name="initial_value">0.0</param>
+      </state_interface>
+      <state_interface name="velocity"/>
+      <state_interface name="effort"/>
+    </joint>
+    <joint name="wheel_rl_joint">
+      <command_interface name="velocity"/>
+      <state_interface name="position">
+        <param name="initial_value">0.0</param>
+      </state_interface>
+      <state_interface name="velocity"/>
+      <state_interface name="effort"/>
+    </joint>
+    <joint name="wheel_rr_joint">
+      <command_interface name="velocity"/>
+      <state_interface name="position">
+        <param name="initial_value">0.0</param>
+      </state_interface>
+      <state_interface name="velocity"/>
+      <state_interface name="effort"/>
+    </joint>
+  </ros2_control>
   <!-- ===== gazebo_ros2_control 插件(驱动 UR 关节) ===== -->
   <gazebo>

Commit message: feat: 同步末端精修相机版本(运行部分快照)
- 源码等价本地基线 1507155:两段式定位(bench 粗定位+腕相机精修,use_refine_detect 默认 false)
- 触觉门控抓取默认路径、GUI 启动竞态三层防御、LLM 任务拆解(规则回退保底)
- 508 tests 全绿,诚实 E2E 通过;运行说明见 README
- 本仓库只含运行相关内容,不含内部过程文档

File: src/lab_cobot_description/urdf/inc/mecanum_base.xacro (robot description, xacro)
@@ -2,6 +2,11 @@
 <!--
   麦克纳姆全向底盘(纯几何,不依赖外部 mesh)。
-  全向运动由 gazebo_ros_planar_move 插件实现(直接对 base 施加 x/y/yaw 速度),
-  轮子为视觉装饰(无 collision,避免与运动学插件冲突)。
+  车体运动来自 wheel_velocity_controller 轮速命令,再由
+  lab_cobot_mecanum_drive pose_from_wheel_commands 按麦轮正解
+  做有界位姿积分并逐 tick SetWorldPose 推进底盘。
+  该模型不声称 Gazebo Classic 中的麦轮滚子接触物理真实:
+  已移除 gazebo_ros_planar_move,但默认推进仍是位姿驱动
+  (非力/速度级物理,底盘不受碰撞阻挡);轮碰撞经 collide_bitmask
+  0x00 禁用,下方滚子摩擦参数为预留配置,当前不生效。
   依赖顶层定义的全局 property: base_length, base_width, base_height, wheel_radius, wheel_width
 -->
@@ -19,11 +24,10 @@
         <material name="base_blue"><color rgba="0.20 0.30 0.60 1.0"/></material>
       </visual>
-      <!-- 碰撞体向下延伸到轮子底部(footprint z=0):轮子无 collision,若仅用车体 box
-           会让 box 底面(footprint z=wheel_radius)贴地、轮子陷入地面 wheel_radius。
-           延伸后 footprint 贴地、轮子接地、车体离地约 wheel_radius(真实底盘外观)。
-           仍是单一 box 碰撞,不引入轮子侧向摩擦,麦轮全向不受影响。 -->
       <collision>
-        <origin xyz="0 0 ${-wheel_radius/2.0}" rpy="0 0 0"/>
-        <geometry><box size="${base_length} ${base_width} ${base_height + wheel_radius}"/></geometry>
+        <geometry><box size="${base_length} ${base_width} ${base_height}"/></geometry>
+      </collision>
+      <collision name="base_ground_support">
+        <origin xyz="0 0 ${-base_z + 0.01}" rpy="0 0 0"/>
+        <geometry><box size="${base_length} ${base_width} 0.02"/></geometry>
       </collision>
       <xacro:box_inertia m="${base_mass}" x="${base_length}" y="${base_width}" z="${base_height}"/>
@@ -34,5 +38,5 @@
       <origin xyz="0 0 ${base_z}" rpy="0 0 0"/>
     </joint>
-    <!-- 4 个麦轮(纯视觉装饰) -->
+    <!-- 4 个麦轮:简化圆柱碰撞 + 视觉滚子条纹 -->
     <xacro:macro name="mec_wheel" params="name x y roller_slant">
       <link name="${name}">
@@ -42,6 +46,9 @@
           <material name="wheel_dark"><color rgba="0.10 0.10 0.10 1.0"/></material>
         </visual>
-        <!-- Side-face roller strips make the wheels read as mecanum in Gazebo/RViz
-             while keeping the wheel collision-free for planar_move. -->
+        <collision>
+          <origin xyz="0 0 0" rpy="${pi/2.0} 0 0"/>
+          <geometry><cylinder radius="${wheel_radius}" length="${wheel_width}"/></geometry>
+        </collision>
+        <!-- Side-face roller strips make the wheels read as mecanum in Gazebo/RViz. -->
         <visual name="${name}_roller_outer_0">
           <origin xyz="0 ${wheel_width/2.0 + 0.003} ${-wheel_radius*0.46}" rpy="0 ${roller_slant*pi/4.0} 0"/>
@@ -102,5 +109,15 @@
         <axis xyz="0 1 0"/>
       </joint>
-      <gazebo reference="${name}"><material>Gazebo/FlatBlack</material></gazebo>
+      <gazebo reference="${name}">
+        <material>Gazebo/FlatBlack</material>
+        <collide_bitmask>0x00</collide_bitmask>
+        <mu1>1.0</mu1>
+        <mu2>0.02</mu2>
+        <fdir1>${cos(roller_slant*pi/4.0)} ${sin(roller_slant*pi/4.0)} 0</fdir1>
+        <kp>1000000.0</kp>
+        <kd>100.0</kd>
+        <maxVel>0.1</maxVel>
+        <minDepth>0.001</minDepth>
+      </gazebo>
     </xacro:macro>
     <xacro:mec_wheel name="wheel_fl" x="${wx}"  y="${wy}"  roller_slant="1"/>
@@ -108,24 +125,4 @@
     <xacro:mec_wheel name="wheel_rl" x="${-wx}" y="${wy}"  roller_slant="-1"/>
     <xacro:mec_wheel name="wheel_rr" x="${-wx}" y="${-wy}" roller_slant="1"/>
-    <!-- 全向驱动插件:订阅 /cmd_vel(Twist 全向),发布 /odom -->
-    <gazebo>
-      <plugin name="gazebo_ros_planar_move" filename="libgazebo_ros_planar_move.so">
-        <ros>
-          <namespace>/</namespace>
-          <remapping>cmd_vel:=cmd_vel</remapping>
-          <remapping>odom:=odom</remapping>
-        </ros>
-        <update_rate>50</update_rate>
-        <publish_rate>50</publish_rate>
-        <publish_odom>true</publish_odom>
-        <!-- EKF 负责发布 odom->base_footprint TF;故此处默认 false -->
-        <publish_odom_tf>${publish_odom_tf}</publish_odom_tf>
-        <odometry_frame>odom</odometry_frame>
-        <robot_base_frame>base_footprint</robot_base_frame>
-        <covariance_x>0.0001</covariance_x>
-        <covariance_y>0.0001</covariance_y>
-        <covariance_yaw>0.01</covariance_yaw>
-      </plugin>
-    </gazebo>
     <gazebo reference="base_link"><material>Gazebo/Blue</material></gazebo>
   </xacro:macro>

File: src/lab_cobot_description/urdf/inc/parallel_gripper.xacro (robot description, xacro)
@@ -2,5 +2,5 @@
 <robot xmlns:xacro="http://www.ros.org/wiki/xacro">
   <!-- Parallel two-finger gripper mounted on the UR tool flange. -->
-  <xacro:macro name="parallel_gripper" params="parent">
+  <xacro:macro name="parallel_gripper" params="parent gazebo_tactile_probe:=false">
     <link name="gripper_base">
       <inertial>
@@ -31,5 +31,5 @@
       <visual>
         <geometry>
-          <box size="0.025 0.012 0.075"/>
+          <box size="0.045 0.012 0.075"/>
         </geometry>
         <material name="gripper_light_grey">
@@ -37,4 +37,16 @@
         </material>
       </visual>
+      <collision>
+        <geometry>
+          <box size="0.045 0.012 0.075"/>
+        </geometry>
+      </collision>
+      <xacro:if value="${gazebo_tactile_probe}">
+        <collision name="gripper_left_finger_tactile_probe">
+          <geometry>
+            <box size="0.045 0.012 0.120"/>
+          </geometry>
+        </collision>
+      </xacro:if>
     </link>
     <joint name="gripper_left_finger_joint" type="prismatic">
@@ -53,5 +65,5 @@
       <visual>
         <geometry>
-          <box size="0.025 0.012 0.075"/>
+          <box size="0.045 0.012 0.075"/>
         </geometry>
         <material name="gripper_light_grey">
@@ -59,4 +71,16 @@
         </material>
       </visual>
+      <collision>
+        <geometry>
+          <box size="0.045 0.012 0.075"/>
+        </geometry>
+      </collision>
+      <xacro:if value="${gazebo_tactile_probe}">
+        <collision name="gripper_right_finger_tactile_probe">
+          <geometry>
+            <box size="0.045 0.012 0.120"/>
+          </geometry>
+        </collision>
+      </xacro:if>
     </link>
     <joint name="gripper_right_finger_joint" type="prismatic">
@@ -73,4 +97,48 @@
       <origin xyz="0 0 0.105" rpy="0 0 0"/>
     </joint>
+    <gazebo reference="gripper_left_finger">
+      <mu1>2.0</mu1>
+      <mu2>2.0</mu2>
+      <kp>1000000.0</kp>
+      <kd>1.0</kd>
+      <minDepth>0.001</minDepth>
+      <maxVel>0.01</maxVel>
+      <sensor name="gripper_left_finger_bumper" type="contact">
+        <always_on>true</always_on>
+        <update_rate>50.0</update_rate>
+        <contact>
+          <collision>gripper_left_finger_tactile_probe_collision_1</collision>
+        </contact>
+        <plugin name="gripper_left_finger_bumper_plugin" filename="libgazebo_ros_bumper.so">
+          <ros>
+            <namespace>/gripper</namespace>
+            <remapping>bumper_states:=left_finger_contacts</remapping>
+          </ros>
+          <frame_name>gripper_left_finger</frame_name>
+        </plugin>
+      </sensor>
+    </gazebo>
+    <gazebo reference="gripper_right_finger">
+      <mu1>2.0</mu1>
+      <mu2>2.0</mu2>
+      <kp>1000000.0</kp>
+      <kd>1.0</kd>
+      <minDepth>0.001</minDepth>
+      <maxVel>0.01</maxVel>
+      <sensor name="gripper_right_finger_bumper" type="contact">
+        <always_on>true</always_on>
+        <update_rate>50.0</update_rate>
+        <contact>
+          <collision>gripper_right_finger_tactile_probe_collision_1</collision>
+        </contact>
+        <plugin name="gripper_right_finger_bumper_plugin" filename="libgazebo_ros_bumper.so">
+          <ros>
+            <namespace>/gripper</namespace>
+            <remapping>bumper_states:=right_finger_contacts</remapping>
+          </ros>
+          <frame_name>gripper_right_finger</frame_name>
+        </plugin>
+      </sensor>
+    </gazebo>
   </xacro:macro>
 </robot>

File: src/lab_cobot_description/urdf/inc/sensors.xacro (robot description, xacro)
@@ -72,9 +72,9 @@
       <xacro:box_inertia m="0.05" x="0.03" y="0.09" z="0.025"/>
     </link>
-    <!-- 装在立柱上方、略高于桌面，向前轻微俯视 station_a 样件 -->
+    <!-- 装在立柱上方侧前方，避开 UR 基座自遮挡并俯视 station_a 样件 -->
     <joint name="camera_joint" type="fixed">
       <parent link="arm_mount_link"/>
       <child link="camera_link"/>
-      <origin xyz="0.10 0 0.35" rpy="0 0.15 0"/>
+      <origin xyz="0.18 -0.22 0.85" rpy="0 0.65 0"/>
     </joint>
     <!-- 光学系(REP-103:z 向前,x 向右,y 向下) -->

File: src/lab_cobot_description/urdf/lab_cobot.urdf.xacro (robot description, xacro)
@@ -3,5 +3,7 @@
   一体化麦轮移动机械臂:麦轮全向底盘 + 基座立柱 + UR5e + 平行夹爪 + 传感器。
   UR5e 用官方 ur_description 的 ur_robot macro(sim_gazebo 模式),装在立柱顶 arm_mount_link。
-  关节由 gazebo_ros2_control 驱动;底盘由 gazebo_ros_planar_move 驱动。
+  关节由 gazebo_ros2_control 驱动;底盘车体运动由 lab_cobot_mecanum_drive 的
+  位姿积分模型(pose_from_wheel_commands,逐 tick SetWorldPose)施加,
+  轮关节旋转仅为视觉同步,不参与推进。
 -->
 <robot xmlns:xacro="http://www.ros.org/wiki/xacro" name="lab_cobot">
@@ -18,4 +20,5 @@
   <xacro:include filename="$(find lab_cobot_description)/urdf/inc/pillar.xacro"/>
   <xacro:include filename="$(find lab_cobot_description)/urdf/inc/sensors.xacro"/>
+  <xacro:include filename="$(find lab_cobot_description)/urdf/inc/wrist_camera.xacro"/>
   <xacro:include filename="$(find lab_cobot_description)/urdf/inc/parallel_gripper.xacro"/>
   <!-- ===== UR5e 参数 ===== -->
@@ -28,8 +31,11 @@
   <xacro:arg name="initial_positions_file" default="$(find lab_cobot_description)/config/initial_positions.yaml"/>
   <xacro:arg name="simulation_controllers" default="$(find lab_cobot_description)/config/lab_cobot_controllers.yaml"/>
+  <xacro:arg name="require_finger_contact" default="false"/>
+  <xacro:arg name="gazebo_tactile_probe" default="false"/>
+  <xacro:arg name="wrist_refine_camera" default="false"/>
   <xacro:property name="initial_positions_file" default="$(arg initial_positions_file)"/>
   <xacro:include filename="$(find ur_description)/urdf/ur_macro.xacro"/>
   <!-- ===== 组装:底盘 → 立柱 → 传感器 ===== -->
-  <!-- base_mass 大幅加重以压低重心、提高抗倾覆(配合臂 home 收拢初始姿态) -->
+  <!-- base_mass 加重以压低重心；Gazebo Classic 麦轮接触仍为近似模型。 -->
   <xacro:mecanum_base base_mass="180.0"/>
   <!-- 立柱降低(0.30)以降低臂安装点与整机重心;仍足够 UR5e 够到 0.75 桌面 -->
@@ -77,5 +83,10 @@
   </xacro:ur_robot>
   <!-- ===== Parallel gripper mounted on UR tool0 ===== -->
-  <xacro:parallel_gripper parent="ur_tool0"/>
+  <xacro:parallel_gripper
+    parent="ur_tool0"
+    gazebo_tactile_probe="$(arg gazebo_tactile_probe)"/>
+  <xacro:if value="$(arg wrist_refine_camera)">
+    <xacro:wrist_refine_camera parent="gripper_base"/>
+  </xacro:if>
   <ros2_control name="gripper_and_wheel_visuals" type="system">
     <hardware>
@@ -137,3 +148,54 @@
     </plugin>
   </gazebo>
+  <gazebo>
+    <plugin name="lab_cobot_mecanum_traction" filename="liblab_cobot_mecanum_drive.so">
+      <control_mode>pose_from_wheel_commands</control_mode>
+      <wheel_command_topic>/wheel_velocity_controller/commands</wheel_command_topic>
+      <base_link>base_link</base_link>
+      <wheel_joint>wheel_fl_joint</wheel_joint>
+      <wheel_joint>wheel_fr_joint</wheel_joint>
+      <wheel_joint>wheel_rl_joint</wheel_joint>
+      <wheel_joint>wheel_rr_joint</wheel_joint>
+      <wheel_radius>${wheel_radius}</wheel_radius>
+      <wheelbase_radius>${base_length/2.0 - wheel_radius + base_width/2.0 + wheel_width/2.0}</wheelbase_radius>
+      <linear_gain>14.0</linear_gain>
+      <angular_gain>24.0</angular_gain>
+      <max_force>2600.0</max_force>
+      <max_torque>1400.0</max_torque>
+      <max_linear_speed>0.45</max_linear_speed>
+      <max_angular_speed>0.9</max_angular_speed>
+      <max_linear_accel>0.8</max_linear_accel>
+      <max_angular_accel>1.5</max_angular_accel>
+      <publish_odom>true</publish_odom>
+      <odom_topic>/odom</odom_topic>
+      <odom_frame>odom</odom_frame>
+      <base_frame>base_footprint</base_frame>
+      <odom_rate>20.0</odom_rate>
+    </plugin>
+  </gazebo>
+  <gazebo>
+    <plugin name="lab_cobot_grasp_fix" filename="liblab_cobot_grasp_fix.so">
+      <object_model>aruco_sample</object_model>
+      <object_link>link</object_link>
+      <tcp_link>gripper_tcp</tcp_link>
+      <left_joint>gripper_left_finger_joint</left_joint>
+      <right_joint>gripper_right_finger_joint</right_joint>
+      <stable_attach_link>ur_wrist_3_link</stable_attach_link>
+      <close_threshold>0.003</close_threshold>
+      <release_threshold>0.003</release_threshold>
+      <grip_count_threshold>1</grip_count_threshold>
+      <require_finger_contact>$(arg require_finger_contact)</require_finger_contact>
+      <contact_count_threshold>1</contact_count_threshold>
+      <max_center_distance>0.090</max_center_distance>
+      <max_abs_x>0.065</max_abs_x>
+      <max_abs_y>0.055</max_abs_y>
+      <min_z>-0.060</min_z>
+      <max_z>0.085</max_z>
+      <grasp_center_offset>-0.037 0.0 0.030</grasp_center_offset>
+      <!-- 约束力保险丝保持默认禁用(0):位姿驱动底盘下正常搬运的
+           fixed-joint ERP 校正力与压桌异常力同量级,阈值不可分离
+           (实测启用会把物块半路丢掉)。压桌爆炸由 place 悬空释放
+           (PLACE_RELEASE_CLEARANCE)机制性根治。 -->
+    </plugin>
+  </gazebo>
 </robot>
