Commit message: feat: 同步 eye-in-hand 检测链与深抓改造(运行部分快照)
- 标准 eye-in-hand:腕相机拍照位检测+顶面 ID=1 marker+Tsai 手眼标定验证探针
- 深抓改造推进:触觉抓取深度收紧+附着期碰撞生命周期修复
- tools 补齐:抓取间隙探针/手眼标定探针/marker 生成/轻量取景器
- 源码等价本地 c29df27,各 commit 均经 build+test 全绿

File: src/lab_cobot_description/urdf/inc/wrist_camera.xacro (robot description, xacro)
@@ -15,5 +15,5 @@
       <parent link="${parent}"/>
       <child link="wrist_camera_link"/>
-      <origin xyz="-0.08 0 0.0" rpy="0 -1.32 0"/>
+      <origin xyz="0.03 0 0.02" rpy="0 ${-pi/2} 0"/>
     </joint>
     <!-- 光学系(REP-103:z 向前,x 向右,y 向下)。 -->
@@ -28,7 +28,7 @@
       <sensor name="wrist_camera" type="depth">
         <always_on>true</always_on>
-        <update_rate>10</update_rate>
+        <update_rate>30</update_rate>
         <camera>
-          <horizontal_fov>1.047</horizontal_fov>
+          <horizontal_fov>1.134464</horizontal_fov>
           <image>
             <width>640</width>
@@ -36,5 +36,5 @@
             <format>R8G8B8</format>
           </image>
-          <clip><near>0.05</near><far>3.0</far></clip>
+          <clip><near>0.01</near><far>3.0</far></clip>
         </camera>
         <plugin name="wrist_camera_plugin" filename="libgazebo_ros_camera.so">
@@ -42,5 +42,5 @@
           <camera_name>wrist_camera</camera_name>
           <frame_name>wrist_camera_optical_frame</frame_name>
-          <min_depth>0.05</min_depth>
+          <min_depth>0.01</min_depth>
           <max_depth>3.0</max_depth>
         </plugin>
