Commit message: fix: 底盘增大与稳定性调整 — 修复遁地/抽搐/频率不统一
- 底盘整体放大：mesh scale 0.001→0.0015，碰撞盒 0.42×0.30×0.12→0.63×0.45×0.18
- 轮径 0.07→0.08，麦轮滚子半径同步增大，悬架安装点外扩并降低
- 修复底盘遁地/抽搐：调整 spawn 高度与悬架连杆参数
- 统一运动频率：Gazebo planar_drive 轮速逆解参数与 URDF 轮径保持一致
- 导航 costmap footprint(0.56×0.62→0.84×0.94)、inflation_radius(0.55→0.80)、robot_radius(0.42→0.60) 同步更新
- 清理已合并的 docs/superpowers 旧计划/设计文档
- bringup/manipulation 配套调整（gripper_driver、mission_node 等）

File: src/lab_cobot_description/urdf/inc/mecanum3_base.xacro (robot description, xacro)
@@ -80,11 +80,46 @@
       <geometry>
         <mesh filename="package://lab_cobot_description/meshes/mecanum3/base_link.stl"
-              scale="0.001 0.001 0.001"/>
+              scale="0.0015 0.0015 0.0015"/>
+      </geometry>
+      <material name="silver"/>
+    </visual>
+    <visual>
+      <origin xyz="0 0 0.0525" rpy="0 0 0"/>
+      <geometry>
+        <box size="0.63 0.18 0.065"/>
+      </geometry>
+      <material name="silver"/>
+    </visual>
+    <visual>
+      <origin xyz="0.275 0.1575 0.0525" rpy="0 0 0"/>
+      <geometry>
+        <box size="0.08 0.135 0.065"/>
+      </geometry>
+      <material name="silver"/>
+    </visual>
+    <visual>
+      <origin xyz="0.275 -0.1575 0.0525" rpy="0 0 0"/>
+      <geometry>
+        <box size="0.08 0.135 0.065"/>
+      </geometry>
+      <material name="silver"/>
+    </visual>
+    <visual>
+      <origin xyz="-0.275 0.1575 0.0525" rpy="0 0 0"/>
+      <geometry>
+        <box size="0.08 0.135 0.065"/>
+      </geometry>
+      <material name="silver"/>
+    </visual>
+    <visual>
+      <origin xyz="-0.275 -0.1575 0.0525" rpy="0 0 0"/>
+      <geometry>
+        <box size="0.08 0.135 0.065"/>
       </geometry>
       <material name="silver"/>
     </visual>
     <collision name="base_simplified_collision">
-      <origin xyz="0 0 0.08" rpy="0 0 0"/>
-      <geometry><box size="0.42 0.30 0.12"/></geometry>
+      <origin xyz="0 0 0.11" rpy="0 0 0"/>
+      <geometry><box size="0.63 0.45 0.18"/></geometry>
     </collision>
   </link>
@@ -141,5 +176,5 @@
       <collision>
         <geometry>
-          <cylinder radius="0.07" length="0.045"/>
+          <cylinder radius="0.08" length="0.045"/>
         </geometry>
       </collision>
@@ -162,5 +197,5 @@
       <collision>
         <geometry>
-          <cylinder radius="0.07" length="0.064"/>
+          <cylinder radius="0.08" length="0.064"/>
         </geometry>
       </collision>
@@ -187,5 +222,5 @@
     parent="base_link"
     child="front_left_arm"
-    xyz="0.020 0.085 0.076"
+    xyz="0.030 0.128 0.020"
     rpy="0 0 ${radians(90)}"/>
   <xacro:mecanum_suspension_joint
@@ -193,5 +228,5 @@
     parent="base_link"
     child="front_right_arm"
-    xyz="0.020 -0.085 0.076"
+    xyz="0.030 -0.128 0.020"
     rpy="0 0 ${radians(90)}"/>
   <xacro:mecanum_suspension_joint
@@ -199,5 +234,5 @@
     parent="base_link"
     child="back_left_arm"
-    xyz="-0.020 0.085 0.076"
+    xyz="-0.030 0.128 0.020"
     rpy="0 0 ${radians(-90)}"/>
   <xacro:mecanum_suspension_joint
@@ -205,5 +240,5 @@
     parent="base_link"
     child="back_right_arm"
-    xyz="-0.020 -0.085 0.076"
+    xyz="-0.030 -0.128 0.020"
     rpy="0 0 ${radians(-90)}"/>
   <!-- Wheels -->
@@ -217,5 +252,5 @@
     parent="front_left_arm"
     child="front_left_wheel_1"
-    xyz="0.03 -0.100 0"
+    xyz="0.045 -0.100 0"
     rpy="0 ${radians(-270)} 0"
     axis_z="-1"/>
@@ -224,5 +259,5 @@
     parent="front_right_arm"
     child="front_right_wheel_1"
-    xyz="-0.03 -0.100 0"
+    xyz="-0.045 -0.100 0"
     rpy="0 ${radians(-90)} 0"
     axis_z="1"/>
@@ -231,5 +266,5 @@
     parent="back_left_arm"
     child="back_left_wheel_1"
-    xyz="-0.03 -0.100 0"
+    xyz="-0.045 -0.100 0"
     rpy="0 ${radians(270)} 0"
     axis_z="-1"/>
@@ -238,5 +273,5 @@
     parent="back_right_arm"
     child="back_right_wheel_1"
-    xyz="0.03 -0.100 0"
+    xyz="0.045 -0.100 0"
     rpy="0 ${radians(90)} 0"
     axis_z="1"/>
@@ -261,5 +296,5 @@
   <joint name="chassis_mount_joint" type="fixed">
     <parent link="base_link"/><child link="chassis_mount_link"/>
-    <origin xyz="0 0 0.165" rpy="0 0 0"/>
+    <origin xyz="0 0 0.248" rpy="0 0 0"/>
   </joint>
   <xacro:macro name="m3_material" params="ref material"><gazebo reference="${ref}"><material>${material}</material></gazebo></xacro:macro>

File: src/lab_cobot_description/urdf/inc/sensors.xacro (robot description, xacro)
@@ -19,5 +19,5 @@
       <parent link="base_link"/>
       <child link="laser"/>
-      <origin xyz="${base_length/2.0 - 0.05} 0 ${base_height/2.0 + 0.04}" rpy="0 0 0"/>
+      <origin xyz="${base_length/2.0 - 0.04} 0 ${base_height/2.0 + 0.04}" rpy="0 0 0"/>
     </joint>
     <gazebo reference="laser">

File: src/lab_cobot_description/urdf/lab_cobot.urdf.xacro (robot description, xacro)
@@ -9,7 +9,7 @@
 <robot xmlns:xacro="http://www.ros.org/wiki/xacro" name="lab_cobot">
   <!-- ===== 全局尺寸(供各部件宏引用) ===== -->
-  <!-- 底盘加宽加长(0.55x0.50):增大支撑多边形,显著提高抗倾覆 -->
-  <xacro:property name="base_length"  value="0.55"/>
-  <xacro:property name="base_width"   value="0.50"/>
+  <!-- 底盘加宽加长(0.83x0.75):1.5× 扩大支撑多边形,显著提高抗倾覆 -->
+  <xacro:property name="base_length"  value="0.63"/>
+  <xacro:property name="base_width"   value="0.45"/>
   <xacro:property name="base_height"  value="0.15"/>
   <xacro:property name="wheel_radius" value="0.08"/>
@@ -173,5 +173,5 @@
     <plugin name="lab_cobot_planar_drive" filename="liblab_cobot_planar_drive.so">
       <wheel_command_topic>/wheel_velocity_controller/commands</wheel_command_topic>
-      <wheel_radius>0.07</wheel_radius>
+      <wheel_radius>0.08</wheel_radius>
       <wheel_separation_width>0.24</wheel_separation_width>
       <wheel_separation_length>0.175</wheel_separation_length>
@@ -180,7 +180,7 @@
       <max_wz>1.2</max_wz>
       <command_timeout>0.3</command_timeout>
-      <chassis_length>0.42</chassis_length>
-      <chassis_width>0.30</chassis_width>
-      <table_safety_margin>0.35</table_safety_margin>
+      <chassis_length>0.63</chassis_length>
+      <chassis_width>0.45</chassis_width>
+      <table_safety_margin>0.30</table_safety_margin>
       <table_a>2.0 1.5 0.8 0.6</table_a>
       <table_b>-2.0 1.5 0.8 0.6</table_b>
