Commit message: mecanum3_chassis_port

File: src/lab_cobot_description/urdf/inc/pillar.xacro (robot description, xacro)
@@ -6,5 +6,5 @@
 -->
 <robot xmlns:xacro="http://www.ros.org/wiki/xacro">
-  <xacro:macro name="base_pillar" params="parent column_height:=0.40 column_size:=0.12 mass:=8.0">
+  <xacro:macro name="base_pillar" params="parent column_height:=0.40 column_size:=0.12 mass:=8.0 mount_offset:=0.0">
     <link name="pillar_link">
       <visual>
@@ -23,5 +23,5 @@
       <parent link="${parent}"/>
       <child link="pillar_link"/>
-      <origin xyz="0 0 ${base_height/2.0}" rpy="0 0 0"/>
+      <origin xyz="0 0 ${mount_offset}" rpy="0 0 0"/>
     </joint>
     <!-- UR 安装点:立柱顶 -->

File: src/lab_cobot_description/urdf/lab_cobot.urdf.xacro (robot description, xacro)
@@ -17,5 +17,5 @@
   <!-- ===== 部件宏 ===== -->
   <xacro:include filename="$(find lab_cobot_description)/urdf/inc/common.xacro"/>
-  <xacro:include filename="$(find lab_cobot_description)/urdf/inc/mecanum_base.xacro"/>
+  <xacro:include filename="$(find lab_cobot_description)/urdf/inc/mecanum3_base.xacro"/>
   <xacro:include filename="$(find lab_cobot_description)/urdf/inc/pillar.xacro"/>
   <xacro:include filename="$(find lab_cobot_description)/urdf/inc/sensors.xacro"/>
@@ -38,7 +38,7 @@
   <!-- ===== 组装:底盘 → 立柱 → 传感器 ===== -->
   <!-- base_mass 加重以压低重心；Gazebo Classic 麦轮接触仍为近似模型。 -->
-  <xacro:mecanum_base base_mass="180.0"/>
+  <xacro:mecanum3_base/>
   <!-- 立柱降低(0.30)以降低臂安装点与整机重心;仍足够 UR5e 够到 0.75 桌面 -->
-  <xacro:base_pillar parent="base_link" column_height="0.30"/>
+  <xacro:base_pillar parent="chassis_mount_link" column_height="0.289" mount_offset="0.0"/>
   <xacro:lab_sensors/>
   <!-- ===== UR5e(装在立柱顶 arm_mount_link;Gazebo 仿真) ===== -->
@@ -109,5 +109,5 @@
       <state_interface name="effort"/>
     </joint>
-    <joint name="wheel_fl_joint">
+    <joint name="front_left_joint">
       <command_interface name="velocity"/>
       <state_interface name="position">
@@ -117,5 +117,5 @@
       <state_interface name="effort"/>
     </joint>
-    <joint name="wheel_fr_joint">
+    <joint name="front_right_joint">
       <command_interface name="velocity"/>
       <state_interface name="position">
@@ -125,5 +125,5 @@
       <state_interface name="effort"/>
     </joint>
-    <joint name="wheel_rl_joint">
+    <joint name="back_left_joint">
       <command_interface name="velocity"/>
       <state_interface name="position">
@@ -133,5 +133,5 @@
       <state_interface name="effort"/>
     </joint>
-    <joint name="wheel_rr_joint">
+    <joint name="back_right_joint">
       <command_interface name="velocity"/>
       <state_interface name="position">
@@ -146,30 +146,4 @@
     <plugin filename="libgazebo_ros2_control.so" name="gazebo_ros2_control">
       <parameters>$(arg simulation_controllers)</parameters>
-    </plugin>
-  </gazebo>
-  <gazebo>
-    <plugin name="lab_cobot_mecanum_traction" filename="liblab_cobot_mecanum_drive.so">
-      <control_mode>pose_from_wheel_commands</control_mode>
-      <wheel_command_topic>/wheel_velocity_controller/commands</wheel_command_topic>
-      <base_link>base_link</base_link>
-      <wheel_joint>wheel_fl_joint</wheel_joint>
-      <wheel_joint>wheel_fr_joint</wheel_joint>
-      <wheel_joint>wheel_rl_joint</wheel_joint>
-      <wheel_joint>wheel_rr_joint</wheel_joint>
-      <wheel_radius>${wheel_radius}</wheel_radius>
-      <wheelbase_radius>${base_length/2.0 - wheel_radius + base_width/2.0 + wheel_width/2.0}</wheelbase_radius>
-      <linear_gain>14.0</linear_gain>
-      <angular_gain>24.0</angular_gain>
-      <max_force>2600.0</max_force>
-      <max_torque>1400.0</max_torque>
-      <max_linear_speed>0.45</max_linear_speed>
-      <max_angular_speed>0.9</max_angular_speed>
-      <max_linear_accel>0.8</max_linear_accel>
-      <max_angular_accel>1.5</max_angular_accel>
-      <publish_odom>true</publish_odom>
-      <odom_topic>/odom</odom_topic>
-      <odom_frame>odom</odom_frame>
-      <base_frame>base_footprint</base_frame>
-      <odom_rate>20.0</odom_rate>
     </plugin>
   </gazebo>

Commit message: feat: 整合底盘链路与多工位导航
- 合并麦轮底盘、Gazebo、导航与真实抓取链既有改动
- 增加单工位导航和固定五工位巡航
- 验证 522 tests 全绿、诚实 A到B E2E、headless 与 GUI 导航演示

File: src/lab_cobot_description/urdf/inc/pillar.xacro (robot description, xacro)
@@ -6,5 +6,5 @@
 -->
 <robot xmlns:xacro="http://www.ros.org/wiki/xacro">
-  <xacro:macro name="base_pillar" params="parent column_height:=0.40 column_size:=0.12 mass:=8.0 mount_offset:=0.0">
+  <xacro:macro name="base_pillar" params="parent column_height:=0.40 column_size:=0.12 mass:=8.0">
     <link name="pillar_link">
       <visual>
@@ -23,5 +23,5 @@
       <parent link="${parent}"/>
       <child link="pillar_link"/>
-      <origin xyz="0 0 ${mount_offset}" rpy="0 0 0"/>
+      <origin xyz="0 0 ${base_height/2.0}" rpy="0 0 0"/>
     </joint>
     <!-- UR 安装点:立柱顶 -->

File: src/lab_cobot_description/urdf/inc/sensors.xacro (robot description, xacro)
@@ -19,5 +19,5 @@
       <parent link="base_link"/>
       <child link="laser"/>
-      <origin xyz="${base_length/2.0 - 0.04} 0 ${base_height/2.0 + 0.04}" rpy="0 0 0"/>
+      <origin xyz="${base_length/2.0 - 0.05} 0 ${base_height/2.0 + 0.04}" rpy="0 0 0"/>
     </joint>
     <gazebo reference="laser">

File: src/lab_cobot_description/urdf/lab_cobot.urdf.xacro (robot description, xacro)
@@ -3,13 +3,13 @@
   一体化麦轮移动机械臂:麦轮全向底盘 + 基座立柱 + UR5e + 平行夹爪 + 传感器。
   UR5e 用官方 ur_description 的 ur_robot macro(sim_gazebo 模式),装在立柱顶 arm_mount_link。
-  底盘视觉轮由 wheel_velocity_controller 驱动；整机位姿由后续/外部
-  mecanum_gazebo_kinematic_drive 节点通过 /set_entity_state 推进。
-  URDF 不再内嵌旧 lab_cobot_mecanum_drive 插件。
+  关节由 gazebo_ros2_control 驱动;底盘车体运动由 lab_cobot_mecanum_drive 的
+  位姿积分模型(pose_from_wheel_commands,逐 tick SetWorldPose)施加,
+  轮关节旋转仅为视觉同步,不参与推进。
 -->
 <robot xmlns:xacro="http://www.ros.org/wiki/xacro" name="lab_cobot">
   <!-- ===== 全局尺寸(供各部件宏引用) ===== -->
-  <!-- 底盘加宽加长(0.83x0.75):1.5× 扩大支撑多边形,显著提高抗倾覆 -->
-  <xacro:property name="base_length"  value="0.63"/>
-  <xacro:property name="base_width"   value="0.45"/>
+  <!-- GitHub main 盒式麦轮底盘。 -->
+  <xacro:property name="base_length"  value="0.55"/>
+  <xacro:property name="base_width"   value="0.50"/>
   <xacro:property name="base_height"  value="0.15"/>
   <xacro:property name="wheel_radius" value="0.08"/>
@@ -17,5 +17,5 @@
   <!-- ===== 部件宏 ===== -->
   <xacro:include filename="$(find lab_cobot_description)/urdf/inc/common.xacro"/>
-  <xacro:include filename="$(find lab_cobot_description)/urdf/inc/mecanum3_base.xacro"/>
+  <xacro:include filename="$(find lab_cobot_description)/urdf/inc/mecanum_base.xacro"/>
   <xacro:include filename="$(find lab_cobot_description)/urdf/inc/pillar.xacro"/>
   <xacro:include filename="$(find lab_cobot_description)/urdf/inc/sensors.xacro"/>
@@ -38,7 +38,7 @@
   <!-- ===== 组装:底盘 → 立柱 → 传感器 ===== -->
   <!-- base_mass 加重以压低重心；Gazebo Classic 麦轮接触仍为近似模型。 -->
-  <xacro:mecanum3_base/>
+  <xacro:mecanum_base base_mass="180.0"/>
   <!-- 立柱降低(0.30)以降低臂安装点与整机重心;仍足够 UR5e 够到 0.75 桌面 -->
-  <xacro:base_pillar parent="chassis_mount_link" column_height="0.289" mount_offset="0.0"/>
+  <xacro:base_pillar parent="base_link" column_height="0.30"/>
   <xacro:lab_sensors/>
   <!-- ===== UR5e(装在立柱顶 arm_mount_link;Gazebo 仿真) ===== -->
@@ -109,53 +109,33 @@
       <state_interface name="effort"/>
     </joint>
-    <joint name="front_left_joint">
-      <command_interface name="velocity"/>
-      <state_interface name="position">
-        <param name="initial_value">0.0</param>
-      </state_interface>
-      <state_interface name="velocity"/>
-      <state_interface name="effort"/>
-    </joint>
-    <joint name="front_right_joint">
-      <command_interface name="velocity"/>
-      <state_interface name="position">
-        <param name="initial_value">0.0</param>
-      </state_interface>
-      <state_interface name="velocity"/>
-      <state_interface name="effort"/>
-    </joint>
-    <joint name="back_left_joint">
-      <command_interface name="velocity"/>
-      <state_interface name="position">
-        <param name="initial_value">0.0</param>
-      </state_interface>
-      <state_interface name="velocity"/>
-      <state_interface name="effort"/>
-    </joint>
-    <joint name="back_right_joint">
-      <command_interface name="velocity"/>
-      <state_interface name="position">
-        <param name="initial_value">0.0</param>
-      </state_interface>
-      <state_interface name="velocity"/>
-      <state_interface name="effort"/>
-    </joint>
-    <joint name="front_left_suspension_joint">
-      <state_interface name="position"/>
-      <state_interface name="velocity"/>
-      <state_interface name="effort"/>
-    </joint>
-    <joint name="front_right_suspension_joint">
-      <state_interface name="position"/>
-      <state_interface name="velocity"/>
-      <state_interface name="effort"/>
-    </joint>
-    <joint name="back_left_suspension_joint">
-      <state_interface name="position"/>
-      <state_interface name="velocity"/>
-      <state_interface name="effort"/>
-    </joint>
-    <joint name="back_right_suspension_joint">
-      <state_interface name="position"/>
+    <joint name="wheel_fl_joint">
+      <command_interface name="velocity"/>
+      <state_interface name="position">
+        <param name="initial_value">0.0</param>
+      </state_interface>
+      <state_interface name="velocity"/>
+      <state_interface name="effort"/>
+    </joint>
+    <joint name="wheel_fr_joint">
+      <command_interface name="velocity"/>
+      <state_interface name="position">
+        <param name="initial_value">0.0</param>
+      </state_interface>
+      <state_interface name="velocity"/>
+      <state_interface name="effort"/>
+    </joint>
+    <joint name="wheel_rl_joint">
+      <command_interface name="velocity"/>
+      <state_interface name="position">
+        <param name="initial_value">0.0</param>
+      </state_interface>
+      <state_interface name="velocity"/>
+      <state_interface name="effort"/>
+    </joint>
+    <joint name="wheel_rr_joint">
+      <command_interface name="velocity"/>
+      <state_interface name="position">
+        <param name="initial_value">0.0</param>
+      </state_interface>
       <state_interface name="velocity"/>
       <state_interface name="effort"/>
@@ -168,21 +148,29 @@
     </plugin>
   </gazebo>
-  <!-- The chassis is a planar kinematic abstraction. Updating it synchronously
-       in Gazebo prevents gravity from fighting an asynchronous pose service. -->
   <gazebo>
-    <plugin name="lab_cobot_planar_drive" filename="liblab_cobot_planar_drive.so">
+    <plugin name="lab_cobot_mecanum_traction" filename="liblab_cobot_mecanum_drive.so">
+      <control_mode>pose_from_wheel_commands</control_mode>
       <wheel_command_topic>/wheel_velocity_controller/commands</wheel_command_topic>
-      <wheel_radius>0.08</wheel_radius>
-      <wheel_separation_width>0.24</wheel_separation_width>
-      <wheel_separation_length>0.175</wheel_separation_length>
-      <max_vx>0.5</max_vx>
-      <max_vy>0.3</max_vy>
-      <max_wz>1.2</max_wz>
-      <command_timeout>0.3</command_timeout>
-      <chassis_length>0.63</chassis_length>
-      <chassis_width>0.45</chassis_width>
-      <table_safety_margin>0.30</table_safety_margin>
-      <table_a>2.0 1.5 0.8 0.6</table_a>
-      <table_b>-2.0 1.5 0.8 0.6</table_b>
+      <base_link>base_link</base_link>
+      <wheel_joint>wheel_fl_joint</wheel_joint>
+      <wheel_joint>wheel_fr_joint</wheel_joint>
+      <wheel_joint>wheel_rl_joint</wheel_joint>
+      <wheel_joint>wheel_rr_joint</wheel_joint>
+      <wheel_radius>${wheel_radius}</wheel_radius>
+      <wheelbase_radius>${base_length/2.0 - wheel_radius + base_width/2.0 + wheel_width/2.0}</wheelbase_radius>
+      <linear_gain>14.0</linear_gain>
+      <angular_gain>24.0</angular_gain>
+      <max_force>2600.0</max_force>
+      <max_torque>1400.0</max_torque>
+      <max_linear_speed>0.45</max_linear_speed>
+      <max_angular_speed>0.9</max_angular_speed>
+      <max_linear_accel>0.8</max_linear_accel>
+      <max_angular_accel>1.5</max_angular_accel>
+      <publish_odom>true</publish_odom>
+      <publish_odom_tf>true</publish_odom_tf>
+      <odom_topic>/odom</odom_topic>
+      <odom_frame>odom</odom_frame>
+      <base_frame>base_footprint</base_frame>
+      <odom_rate>20.0</odom_rate>
     </plugin>
   </gazebo>
