Commit message: fix: 抗倾覆改造 - 底盘加大至0.55x0.50+加重180kg+降柱0.30+臂home收拢初始姿态;移除Gazebo Classic不支持的spawn -J

File: src/lab_cobot_description/urdf/lab_cobot.urdf.xacro (robot description, xacro)
@@ -7,6 +7,7 @@
 <robot xmlns:xacro="http://www.ros.org/wiki/xacro" name="lab_cobot">
   <!-- ===== 全局尺寸(供各部件宏引用) ===== -->
-  <xacro:property name="base_length"  value="0.50"/>
-  <xacro:property name="base_width"   value="0.36"/>
+  <!-- 底盘加宽加长(0.55x0.50):增大支撑多边形,显著提高抗倾覆 -->
+  <xacro:property name="base_length"  value="0.55"/>
+  <xacro:property name="base_width"   value="0.50"/>
   <xacro:property name="base_height"  value="0.15"/>
   <xacro:property name="wheel_radius" value="0.08"/>
@@ -25,11 +26,13 @@
   <xacro:arg name="physical_params" default="$(find ur_description)/config/$(arg ur_type)/physical_parameters.yaml"/>
   <xacro:arg name="visual_params" default="$(find ur_description)/config/$(arg ur_type)/visual_parameters.yaml"/>
-  <xacro:arg name="initial_positions_file" default="$(find ur_description)/config/initial_positions.yaml"/>
+  <xacro:arg name="initial_positions_file" default="$(find lab_cobot_description)/config/initial_positions.yaml"/>
   <xacro:arg name="simulation_controllers" default="$(find lab_cobot_description)/config/lab_cobot_controllers.yaml"/>
   <xacro:property name="initial_positions_file" default="$(arg initial_positions_file)"/>
   <xacro:include filename="$(find ur_description)/urdf/ur_macro.xacro"/>
   <!-- ===== 组装:底盘 → 立柱 → 传感器 ===== -->
-  <xacro:mecanum_base/>
-  <xacro:base_pillar parent="base_link" column_height="0.40"/>
+  <!-- base_mass 大幅加重以压低重心、提高抗倾覆(配合臂 home 收拢初始姿态) -->
+  <xacro:mecanum_base base_mass="180.0"/>
+  <!-- 立柱降低(0.30)以降低臂安装点与整机重心;仍足够 UR5e 够到 0.75 桌面 -->
+  <xacro:base_pillar parent="base_link" column_height="0.30"/>
   <xacro:lab_sensors/>
   <!-- ===== UR5e(装在立柱顶 arm_mount_link;Gazebo 仿真) ===== -->
