Commit message: fix: publish real suspension joint states

File: src/lab_cobot_description/urdf/lab_cobot.urdf.xacro (robot description, xacro)
@@ -141,4 +141,24 @@
       <state_interface name="effort"/>
     </joint>
+    <joint name="front_left_suspension_joint">
+      <state_interface name="position"/>
+      <state_interface name="velocity"/>
+      <state_interface name="effort"/>
+    </joint>
+    <joint name="front_right_suspension_joint">
+      <state_interface name="position"/>
+      <state_interface name="velocity"/>
+      <state_interface name="effort"/>
+    </joint>
+    <joint name="back_left_suspension_joint">
+      <state_interface name="position"/>
+      <state_interface name="velocity"/>
+      <state_interface name="effort"/>
+    </joint>
+    <joint name="back_right_suspension_joint">
+      <state_interface name="position"/>
+      <state_interface name="velocity"/>
+      <state_interface name="effort"/>
+    </joint>
   </ros2_control>
   <!-- ===== gazebo_ros2_control 插件(驱动 UR 关节) ===== -->

Commit message: feat: add multiple manipulation tasks and validation

File: src/lab_cobot_description/urdf/lab_cobot.urdf.xacro (robot description, xacro)
@@ -36,5 +36,10 @@
   <xacro:arg name="enable_lab_sensors" default="true"/>
   <xacro:arg name="wrist_refine_camera" default="false"/>
+  <xacro:arg name="tube_insert_fixed_base" default="false"/>
   <xacro:property name="initial_positions_file" default="$(arg initial_positions_file)"/>
+  <xacro:property name="mecanum_control_mode" value="pose_from_wheel_commands"/>
+  <xacro:if value="$(arg tube_insert_fixed_base)">
+    <xacro:property name="mecanum_control_mode" value="fixed_pose"/>
+  </xacro:if>
   <xacro:include filename="$(find ur_description)/urdf/ur_macro.xacro"/>
   <!-- ===== 组装:底盘 → 立柱 → 传感器 ===== -->
@@ -154,5 +159,5 @@
   <gazebo>
     <plugin name="lab_cobot_mecanum_traction" filename="liblab_cobot_mecanum_drive.so">
-      <control_mode>pose_from_wheel_commands</control_mode>
+      <control_mode>${mecanum_control_mode}</control_mode>
       <wheel_command_topic>/wheel_velocity_controller/commands</wheel_command_topic>
       <base_link>base_link</base_link>
@@ -182,6 +187,6 @@
     <plugin name="lab_cobot_grasp_fix" filename="liblab_cobot_grasp_fix.so">
       <object_model>aruco_sample</object_model>
+      <object_model>tooling_fixture_box</object_model>
       <object_model>tooling_hand_tools</object_model>
-      <object_model>tooling_fixture_box</object_model>
       <object_model>board_test_fixture</object_model>
       <object_model>high_voltage_probe_kit</object_model>
@@ -196,4 +201,5 @@
       <object_model>test_tube_8</object_model>
       <object_model>test_tube_9</object_model>
+      <object_model>material_cube_yellow</object_model>
       <object_link>link</object_link>
       <tcp_link>gripper_tcp</tcp_link>
